Commit message: feat: add vision-guided bottle pick-shake-place pipeline

File: src/hv_arm/urdf/gazebo.xacro (robot description, xacro)
@@ -12,3 +12,20 @@
       </plugin>
   </gazebo>
+  <!-- Physically connects the bottle to the robot during grasping -->
+  <gazebo>
+    <plugin
+      filename="gz-sim-detachable-joint-system"
+      name="gz::sim::systems::DetachableJoint">
+      <!-- Moving physics link belonging to the Panda model -->
+      <parent_link>panda_link7</parent_link>
+      <!-- Gazebo model and link defined in empty.world -->
+      <child_model>bottle</child_model>
+      <child_link>bottle_link</child_link>
+      <!-- Runtime command topics -->
+      <detach_topic>/bottle/detach</detach_topic>
+      <attach_topic>/bottle/attach</attach_topic>
+      <!-- Reports whether the fixed joint exists -->
+      <output_topic>/bottle/attachment_state</output_topic>
+    </plugin>
+  </gazebo>
 </robot>

File: src/hv_arm/urdf/sensors.xacro (robot description, xacro)
@@ -23,5 +23,5 @@
     </link>
     <joint name="camera_joint" type="fixed">
-        <origin xyz="0.6 0 1.0" rpy="0.0 0.0 0.0"/>
+        <origin xyz="0.6 0 1.0" rpy="0 ${pi/2} 0"/>
         <parent link="panda_link0"/>
         <child link="camera_link"/>
@@ -35,5 +35,5 @@
     <gazebo reference="camera_link">
         <sensor name="camera" type="camera">
-            <pose>0 0 0 0 1.57 0</pose>
+            <pose>0 0 0 0 0 0</pose>
             <visualize>true</visualize>
             <update_rate>10.0</update_rate>
